File: XS3868-Shield.sch (KiCad schematic (older format))
At the start: 6 parts, among them P1 CONN_01X03, P2 CONN_01X02, U1 XS3868, U2 AP111733

Commit message: Layout review
Parts:
- added C3: 100u, SMD_Packages:SMD-2512_Pol, symbol CP1_Small
- added U3: LM7805, RACE_UP_ED:LM7805_TO92, symbol LM7805
- C1, C2: footprint Capacitors_SMD:C_1206_HandSoldering -> SMD_Packages:SMD-2512_Pol
Connections:
- net +12V: now also U3.VI; no longer U2.3 (VI)
- net +3V3: now also C3.1; no longer C2.1
- net GND: now also C3.2, U3.GND
- new net +5V: C2.1, U2.3 (VI), U3.VO
Other:
- moved on the sheet: U2
Changed lines of the file:
@@
 L AP111733 U2
 U 1 1 58AEE048
-P 6450 3150
-F 0 "U2" H 6450 3517 50  0000 C CNN
-F 1 "AP111733" H 6450 3426 50  0000 C CNN
-F 2 "TO_SOT_Packages_SMD:SOT-223" H 6450 2800 50  0001 C CNN
-F 3 "" H 6550 2900 50  0000 C CNN
-	1    6450 3150
+P 7625 3150
+F 0 "U2" H 7625 3517 50  0000 C CNN
+F 1 "AP111733" H 7625 3426 50  0000 C CNN
+F 2 "TO_SOT_Packages_SMD:SOT-223" H 7625 2800 50  0001 C CNN
+F 3 "" H 7725 2900 50  0000 C CNN
+	1    7625 3150
 	1    0    0    -1
 $EndComp
@@
 F 0 "C2" H 7141 3396 50  0000 L CNN
 F 1 "100u" H 7141 3305 50  0000 L CNN
-F 2 "Capacitors_SMD:C_1206_HandSoldering" H 7050 3350 50  0001 C CNN
+F 2 "SMD_Packages:SMD-2512_Pol" H 7050 3350 50  0001 C CNN
 F 3 "" H 7050 3350 50  0000 C CNN
 	1    7050 3350
@@
 F 0 "C1" H 5891 3396 50  0000 L CNN
 F 1 "100u" H 5891 3305 50  0000 L CNN
-F 2 "Capacitors_SMD:C_1206_HandSoldering" H 5800 3350 50  0001 C CNN
+F 2 "SMD_Packages:SMD-2512_Pol" H 5800 3350 50  0001 C CNN
 F 3 "" H 5800 3350 50  0000 C CNN
 	1    5800 3350
@@
 $Comp
 L +3.3V #PWR06
-U 1 1 58AEE6DA
-P 7050 3100
-F 0 "#PWR06" H 7050 2950 50  0001 C CNN
-F 1 "+3.3V" H 7065 3273 50  0000 C CNN
-F 2 "" H 7050 3100 50  0000 C CNN
-F 3 "" H 7050 3100 50  0000 C CNN
-	1    7050 3100
-	1    0    0    -1
-$EndComp
-$Comp
-L +3.3V #PWR07
 U 1 1 58AEE722
 P 4950 5350
-F 0 "#PWR07" H 4950 5200 50  0001 C CNN
+F 0 "#PWR06" H 4950 5200 50  0001 C CNN
 F 1 "+3.3V" V 4965 5478 50  0000 L CNN
 F 2 "" H 4950 5350 50  0000 C CNN
@@
 	1    4950 5350
 	0    -1   -1   0
+$EndComp
+$Comp
+L LM7805 U3
+U 1 1 58C2C571
+P 6450 3200
+F 0 "U3" H 6600 3004 50  0000 C CNN
+F 1 "LM7805" H 6450 3400 50  0000 C CNN
+F 2 "RACE_UP_ED:LM7805_TO92" H 6450 3200 50  0001 C CNN
+F 3 "" H 6450 3200 50  0000 C CNN
+	1    6450 3200
+	1    0    0    -1
+$EndComp
+$Comp
+L +3.3V #PWR07
+U 1 1 58C2C7B9
+P 8100 3100
+F 0 "#PWR07" H 8100 2950 50  0001 C CNN
+F 1 "+3.3V" H 8115 3273 50  0000 C CNN
+F 2 "" H 8100 3100 50  0000 C CNN
+F 3 "" H 8100 3100 50  0000 C CNN
+	1    8100 3100
+	1    0    0    -1
+$EndComp
+$Comp
+L CP1_Small C3
+U 1 1 58C2C857
+P 8100 3350
+F 0 "C3" H 8191 3396 50  0000 L CNN
+F 1 "100u" H 8191 3305 50  0000 L CNN
+F 2 "SMD_Packages:SMD-2512_Pol" H 8100 3350 50  0001 C CNN
+F 3 "" H 8100 3350 50  0000 C CNN
+	1    8100 3350
+	1    0    0    -1
+$EndComp
+$Comp
+L +5V #PWR08
+U 1 1 58C2C948
+P 7050 3100
+F 0 "#PWR08" H 7050 2950 50  0001 C CNN
+F 1 "+5V" H 7050 3240 50  0000 C CNN
+F 2 "" H 7050 3100 50  0000 C CNN
+F 3 "" H 7050 3100 50  0000 C CNN
+	1    7050 3100
+	1    0    0    -1
 $EndComp
 Wire Wire Line
@@
 	5800 3100 5800 3250
 Wire Wire Line
-	5800 3150 6150 3150
-Wire Wire Line
 	7050 3100 7050 3250
-Wire Wire Line
-	7050 3150 6750 3150
 Wire Wire Line
 	5800 3450 5800 3500
 Wire Wire Line
-	5800 3500 7050 3500
+	5800 3500 8100 3500
 Wire Wire Line
 	7050 3500 7050 3450
@@
 Wire Wire Line
 	5250 3350 5150 3350
+Wire Wire Line
+	7925 3150 8100 3150
+Wire Wire Line
+	8100 3100 8100 3250
+Connection ~ 8100 3150
+Wire Wire Line
+	8100 3500 8100 3450
+Connection ~ 7050 3500
+Wire Wire Line
+	7625 3450 7625 3500
+Connection ~ 7625 3500
+Wire Wire Line
+	5800 3150 6050 3150
+Wire Wire Line
+	6850 3150 7325 3150
 $EndSCHEMATC
